Commit message: gazebo-URDF

File: kyun_description/urdf/kyun.urdf (robot description, URDF)
Before this commit: robot kyun, 7 links, 6 joints
Links:
- link 2nd_link: geometry collision mesh filename=package://kyun_description/mesh/frame12.stl scale=0.001 0.001 0.001; visual mesh filename=package://kyun_description/mesh/frame12.stl scale=0.001 0.001 0.001
- link 3rd_link: geometry collision mesh filename=package://kyun_description/mesh/servo02.stl scale=0.001 0.001 0.001; visual mesh filename=package://kyun_description/mesh/servo02.stl scale=0.001 0.001 0.001
- link 4th_link: geometry collision mesh filename=package://kyun_description/mesh/servo03.stl scale=0.001 0.001 0.001; visual mesh filename=package://kyun_description/mesh/servo03.stl scale=0.001 0.001 0.001
- link 5th_link: geometry collision mesh filename=package://kyun_description/mesh/servo04.stl scale=0.001 0.001 0.001; visual mesh filename=package://kyun_description/mesh/servo04.stl scale=0.001 0.001 0.001
- link 6th_link: geometry collision mesh filename=package://kyun_description/mesh/frame13.stl scale=0.001 0.001 0.001; visual mesh filename=package://kyun_description/mesh/frame13.stl scale=0.001 0.001 0.001
- link base_link: geometry collision mesh filename=package://kyun_description/mesh/servo01.stl scale=0.001 0.001 0.001; visual mesh filename=package://kyun_description/mesh/servo01.stl scale=0.001 0.001 0.001
Joints:
- removed joint base_link_joint
- added joint world_to_base: type fixed, parent world, child base_link, origin xyz=0 0 0
