Commit message: workgit add -A

File: kyun_description/urdf/kyun_simple_work.xacro (robot description, xacro)
@@ -25,15 +25,26 @@
   </inertial>
 </link>
-<joint name="base_to_2nd" type="continuous">
+<joint name="base_to_second" type="continuous">
   <parent link="base_link"/>
-  <child link="2nd_link"/>
+  <child link="second_link"/>
   <origin xyz="0 0 0" rpy="0 0 0"/>
   <axis xyz="0 0 1"/>
-  <dynamics damping="0.1"/>
+  <dynamics damping="0.7"/>
 </joint>
-<link name="2nd_link">
+<transmission name="base_trans">
+    <type>transmission_interface/SimpleTransmission</type>
+    <joint name="base_to_second">
+      <hardwareInterface>hardware_interface/EffortJointInterface</hardwareInterface>
+    </joint>
+    <actuator name="base_motor">
+       <hardwareInterface>hardware_interface/EffortJointInterface</hardwareInterface>
+       <mechanismReduction>1</mechanismReduction>
+    </actuator>
+</transmission>
+<link name="second_link">
   <visual>
     <geometry>
       <mesh filename="package://kyun_description/mesh/frame12.stl" scale="0.001 0.001 0.001"/>
+      <origin xyz="0 0 0"/>
     </geometry>
   </visual>
@@ -41,10 +52,51 @@
     <geometry>
       <mesh filename="package://kyun_description/mesh/frame12.stl" scale="0.001 0.001 0.001"/>
+      <origin xyz="0 0 0"/>
     </geometry>
   </collision>
   <inertial>
-    <mass value="0.6"/>
-    <inertia ixx="1e-3" ixy="0" ixz="0" iyy="1e-3" iyz="0" izz="1e-3"/>
+    <mass value="0.0228"/>
+    <inertia ixx="0.012587" ixy="0" ixz="0" iyy="0.009052" iyz="0" izz="0.010677"/>
   </inertial>
 </link>
+<joint name="second_to_third" type="continuous">
+  <parent link="second_link"/>
+  <child link="third_link"/>
+  <origin xyz="-0.00963 0.019 0.05" rpy="0 0 0"/>
+  <axis xyz="0 1 0"/>
+  <dynamics damping="0.7"/>
+</joint>
+<transmission name="second_trans">
+    <type>transmission_interface/SimpleTransmission</type>
+    <joint name="second_to_third">
+      <hardwareInterface>hardware_interface/EffortJointInterface</hardwareInterface>
+    </joint>
+    <actuator name="second_motor">
+       <hardwareInterface>hardware_interface/EffortJointInterface</hardwareInterface>
+       <mechanismReduction>1</mechanismReduction>
+    </actuator>
+</transmission>
+<link name="third_link">
+  <visual>
+    <geometry>
+      <mesh filename="package://kyun_description/mesh/servo02.stl" scale="0.001 0.001 0.001"/>
+    </geometry>
+  </visual>
+  <collision>
+    <geometry>
+      <mesh filename="package://kyun_description/mesh/servo02.stl" scale="0.001 0.001 0.001"/>
+    </geometry>
+  </collision>
+  <inertial>
+    <mass value="0.0638"/>
+    <inertia ixx="0.021267" ixy="0" ixz="0" iyy="0.020277" iyz="0" izz="0.011317"/>
+  </inertial>
+</link>
+<gazebo>
+  <plugin name="gazebo_ros_control" filename="libgazebo_ros_control.so">
+    <robotNamespace>/kyun_simple_work</robotNamespace>
+    <robotSimType>gazebo_ros_control/DefaultRobotHWSim</robotSimType>
+    <legacyModeNS>true</legacyModeNS>
+  </plugin>
+</gazebo>
 </robot>

Commit message: gravity

File: kyun_description/urdf/kyun_simple_work.xacro (robot description, xacro)
@@ -25,14 +25,15 @@
   </inertial>
 </link>
-<joint name="base_to_second" type="continuous">
+<joint name="base_to_2nd" type="revolute">
   <parent link="base_link"/>
-  <child link="second_link"/>
+  <child link="2nd_link"/>
   <origin xyz="0 0 0" rpy="0 0 0"/>
   <axis xyz="0 0 1"/>
   <dynamics damping="0.7"/>
+  <limit lower="-1.5" upper="1.5" effort="0" velocity="0"/>
 </joint>
 <transmission name="base_trans">
     <type>transmission_interface/SimpleTransmission</type>
-    <joint name="base_to_second">
+    <joint name="base_to_2nd">
       <hardwareInterface>hardware_interface/EffortJointInterface</hardwareInterface>
     </joint>
@@ -42,5 +43,5 @@
     </actuator>
 </transmission>
-<link name="second_link">
+<link name="2nd_link">
   <visual>
     <geometry>
@@ -57,28 +58,30 @@
   <inertial>
     <mass value="0.0228"/>
-    <inertia ixx="0.012587" ixy="0" ixz="0" iyy="0.009052" iyz="0" izz="0.010677"/>
-  </inertial>
-</link>
-<joint name="second_to_third" type="continuous">
-  <parent link="second_link"/>
-  <child link="third_link"/>
+    <inertia ixx="0.0012587" ixy="0" ixz="0" iyy="0.0009052" iyz="0" izz="0.0010677"/>
+  </inertial>
+</link>
+<joint name="2nd_to_3rd" type="revolute">
+  <parent link="2nd_link"/>
+  <child link="3rd_link"/>
   <origin xyz="-0.00963 0.019 0.05" rpy="0 0 0"/>
   <axis xyz="0 1 0"/>
   <dynamics damping="0.7"/>
-</joint>
-<transmission name="second_trans">
-    <type>transmission_interface/SimpleTransmission</type>
-    <joint name="second_to_third">
-      <hardwareInterface>hardware_interface/EffortJointInterface</hardwareInterface>
-    </joint>
-    <actuator name="second_motor">
-       <hardwareInterface>hardware_interface/EffortJointInterface</hardwareInterface>
-       <mechanismReduction>1</mechanismReduction>
-    </actuator>
-</transmission>
-<link name="third_link">
+  <limit lower="-1.5" upper="1.5" effort="0" velocity="0"/>
+</joint>
+<transmission name="2nd_trans">
+    <type>transmission_interface/SimpleTransmission</type>
+    <joint name="2nd_to_3rd">
+      <hardwareInterface>hardware_interface/EffortJointInterface</hardwareInterface>
+    </joint>
+    <actuator name="2nd_motor">
+       <hardwareInterface>hardware_interface/EffortJointInterface</hardwareInterface>
+       <mechanismReduction>1</mechanismReduction>
+    </actuator>
+</transmission>
+<link name="3rd_link">
   <visual>
     <geometry>
       <mesh filename="package://kyun_description/mesh/servo02.stl" scale="0.001 0.001 0.001"/>
+      <origin xyz="0 0 0"/>
     </geometry>
   </visual>
@@ -86,9 +89,112 @@
     <geometry>
       <mesh filename="package://kyun_description/mesh/servo02.stl" scale="0.001 0.001 0.001"/>
+      <origin xyz="0 0 0"/>
     </geometry>
   </collision>
   <inertial>
     <mass value="0.0638"/>
-    <inertia ixx="0.021267" ixy="0" ixz="0" iyy="0.020277" iyz="0" izz="0.011317"/>
+    <inertia ixx="0.0021267" ixy="0" ixz="0" iyy="0.0020277" iyz="0" izz="0.0011317"/>
+  </inertial>
+</link>
+<joint name="3rd_to_4th" type="revolute">
+  <parent link="3rd_link"/>
+  <child link="4th_link"/>
+  <origin xyz="0.019 -0.018 0.06075" rpy="0 0 0"/>
+  <axis xyz="1 0 0"/>
+  <dynamics damping="0.7"/>
+  <limit lower="-1.5" upper="1.5" effort="0" velocity="0"/>
+</joint>
+<transmission name="3rd_trans">
+    <type>transmission_interface/SimpleTransmission</type>
+    <joint name="3rd_to_4th">
+      <hardwareInterface>hardware_interface/EffortJointInterface</hardwareInterface>
+    </joint>
+    <actuator name="3rd_motor">
+       <hardwareInterface>hardware_interface/EffortJointInterface</hardwareInterface>
+       <mechanismReduction>1</mechanismReduction>
+    </actuator>
+</transmission>
+<link name="4th_link">
+  <visual>
+    <geometry>
+      <mesh filename="package://kyun_description/mesh/servo03.stl" scale="0.001 0.001 0.001"/>
+    </geometry>
+  </visual>
+  <collision>
+    <geometry>
+      <mesh filename="package://kyun_description/mesh/servo03.stl" scale="0.001 0.001 0.001"/>
+    </geometry>
+  </collision>
+  <inertial>
+    <mass value="0.099806"/>
+    <inertia ixx="0.0028791" ixy="0" ixz="0" iyy="0.0028648" iyz="0" izz="0.0021805"/>
+  </inertial>
+</link>
+<joint name="4th_to_5th" type="revolute">
+  <parent link="4th_link"/>
+  <child link="5th_link"/>
+  <origin xyz="-0.019 -0.02 0.024" rpy="0 0 0"/>
+  <axis xyz="0 1 0"/>
+  <dynamics damping="0.7"/>
+  <limit lower="-1.5" upper="1.5" effort="0" velocity="0"/>
+</joint>
+<transmission name="4th_trans">
+    <type>transmission_interface/SimpleTransmission</type>
+    <joint name="4th_to_5th">
+      <hardwareInterface>hardware_interface/EffortJointInterface</hardwareInterface>
+    </joint>
+    <actuator name="4th_motor">
+       <hardwareInterface>hardware_interface/EffortJointInterface</hardwareInterface>
+       <mechanismReduction>1</mechanismReduction>
+    </actuator>
+</transmission>
+<link name="5th_link">
+  <visual>
+    <geometry>
+      <mesh filename="package://kyun_description/mesh/servo04.stl" scale="0.001 0.001 0.001"/>
+    </geometry>
+  </visual>
+  <collision>
+    <geometry>
+      <mesh filename="package://kyun_description/mesh/servo04.stl" scale="0.001 0.001 0.001"/>
+    </geometry>
+  </collision>
+  <inertial>
+    <mass value="0.063759"/>
+    <inertia ixx="0.0020277" ixy="0" ixz="0" iyy="0.0021267" iyz="0" izz="0.0011317"/>
+  </inertial>
+</link>
+<joint name="5th_to_6th" type="revolute">
+  <parent link="5th_link"/>
+  <child link="6th_link"/>
+  <origin xyz="0.0205 0.02 0.06075" rpy="0 0 0"/>
+  <axis xyz="1 0 0"/>
+  <dynamics damping="0.7"/>
+  <limit lower="-1.5" upper="1.5" effort="0" velocity="0"/>
+</joint>
+<transmission name="5th_trans">
+    <type>transmission_interface/SimpleTransmission</type>
+    <joint name="5th_to_6th">
+      <hardwareInterface>hardware_interface/EffortJointInterface</hardwareInterface>
+    </joint>
+    <actuator name="5th_motor">
+       <hardwareInterface>hardware_interface/EffortJointInterface</hardwareInterface>
+       <mechanismReduction>1</mechanismReduction>
+    </actuator>
+</transmission>
+<link name="6th_link">
+  <visual>
+    <geometry>
+      <mesh filename="package://kyun_description/mesh/frame13.stl" scale="0.001 0.001 0.001"/>
+    </geometry>
+  </visual>
+  <collision>
+    <geometry>
+      <mesh filename="package://kyun_description/mesh/frame13.stl" scale="0.001 0.001 0.001"/>
+    </geometry>
+  </collision>
+  <inertial>
+    <mass value="0.059571"/>
+    <inertia ixx="0.0011416" ixy="0" ixz="0" iyy="0.0011103" iyz="0" izz="0.0020421"/>
   </inertial>
 </link>

Commit message: completion

File: kyun_description/urdf/kyun_simple_work.xacro (robot description, xacro)
@@ -1,4 +1,10 @@
 <?xml version="1.0"?>
-<robot name="kyun" xmlns:xacro="http://www.ros.org/wiki/xacro">
+<robot name="kyun_simple_work" xmlns:xacro="http://www.ros.org/wiki/xacro">
+<material name="gray">
+  <color rgba="0.5 0.5 0.5 2.5"/>
+</material>
+<material name="white">
+  <color rgba="1.0 1.0 1.0 1"/>
+</material>
 <link name="world"/>
 <joint name="world_to_base" type="fixed">
@@ -13,4 +19,5 @@
       <origin xyz="0 0 0.0465"/>
     </geometry>
+    <material name="gray"/>
   </visual>
   <collision>
@@ -25,4 +32,7 @@
   </inertial>
 </link>
+<gazebo reference="base_link">
+  <material>Gazebo/Grey</material>
+</gazebo>
 <joint name="base_to_2nd" type="revolute">
   <parent link="base_link"/>
@@ -31,5 +41,5 @@
   <axis xyz="0 0 1"/>
   <dynamics damping="0.7"/>
-  <limit lower="-1.5" upper="1.5" effort="0" velocity="0"/>
+  <limit lower="-1.5" upper="1.5" effort="0.5" velocity="6.0"/>
 </joint>
 <transmission name="base_trans">
@@ -39,6 +49,6 @@
     </joint>
     <actuator name="base_motor">
-       <hardwareInterface>hardware_interface/EffortJointInterface</hardwareInterface>
-       <mechanismReduction>1</mechanismReduction>
+      <hardwareInterface>hardware_interface/EffortJointInterface</hardwareInterface>
+      <mechanismReduction>1</mechanismReduction>
     </actuator>
 </transmission>
@@ -49,4 +59,5 @@
       <origin xyz="0 0 0"/>
     </geometry>
+    <material name="grey"/>
   </visual>
   <collision>
@@ -61,4 +72,7 @@
   </inertial>
 </link>
+<gazebo reference="2nd_link">
+  <material>Gazebo/Grey</material>
+</gazebo>
 <joint name="2nd_to_3rd" type="revolute">
   <parent link="2nd_link"/>
@@ -67,5 +81,5 @@
   <axis xyz="0 1 0"/>
   <dynamics damping="0.7"/>
-  <limit lower="-1.5" upper="1.5" effort="0" velocity="0"/>
+  <limit lower="-1.5" upper="1.5" effort="0.5" velocity="6.0"/>
 </joint>
 <transmission name="2nd_trans">
@@ -75,6 +89,6 @@
     </joint>
     <actuator name="2nd_motor">
-       <hardwareInterface>hardware_interface/EffortJointInterface</hardwareInterface>
-       <mechanismReduction>1</mechanismReduction>
+      <hardwareInterface>hardware_interface/EffortJointInterface</hardwareInterface>
+      <mechanismReduction>1</mechanismReduction>
     </actuator>
 </transmission>
@@ -85,4 +99,5 @@
       <origin xyz="0 0 0"/>
     </geometry>
+    <material name="grey"/>
   </visual>
   <collision>
@@ -97,4 +112,7 @@
   </inertial>
 </link>
+<gazebo reference="3rd_link">
+  <material>Gazebo/Grey</material>
+</gazebo>
 <joint name="3rd_to_4th" type="revolute">
   <parent link="3rd_link"/>
@@ -103,5 +121,5 @@
   <axis xyz="1 0 0"/>
   <dynamics damping="0.7"/>
-  <limit lower="-1.5" upper="1.5" effort="0" velocity="0"/>
+  <limit lower="-1.5" upper="1.5" effort="0.5" velocity="6.0"/>
 </joint>
 <transmission name="3rd_trans">
@@ -111,6 +129,6 @@
     </joint>
     <actuator name="3rd_motor">
-       <hardwareInterface>hardware_interface/EffortJointInterface</hardwareInterface>
-       <mechanismReduction>1</mechanismReduction>
+      <hardwareInterface>hardware_interface/EffortJointInterface</hardwareInterface>
+      <mechanismReduction>1</mechanismReduction>
     </actuator>
 </transmission>
@@ -120,4 +138,5 @@
       <mesh filename="package://kyun_description/mesh/servo03.stl" scale="0.001 0.001 0.001"/>
     </geometry>
+    <material name="grey"/>
   </visual>
   <collision>
@@ -131,4 +150,7 @@
   </inertial>
 </link>
+<gazebo reference="4th_link">
+  <material>Gazebo/Grey</material>
+</gazebo>
 <joint name="4th_to_5th" type="revolute">
   <parent link="4th_link"/>
@@ -137,5 +159,5 @@
   <axis xyz="0 1 0"/>
   <dynamics damping="0.7"/>
-  <limit lower="-1.5" upper="1.5" effort="0" velocity="0"/>
+  <limit lower="-1.5" upper="1.5" effort="0.5" velocity="6.0"/>
 </joint>
 <transmission name="4th_trans">
@@ -145,6 +167,6 @@
     </joint>
     <actuator name="4th_motor">
-       <hardwareInterface>hardware_interface/EffortJointInterface</hardwareInterface>
-       <mechanismReduction>1</mechanismReduction>
+      <hardwareInterface>hardware_interface/EffortJointInterface</hardwareInterface>
+      <mechanismReduction>1</mechanismReduction>
     </actuator>
 </transmission>
@@ -154,4 +176,5 @@
       <mesh filename="package://kyun_description/mesh/servo04.stl" scale="0.001 0.001 0.001"/>
     </geometry>
+    <material name="grey"/>
   </visual>
   <collision>
@@ -165,4 +188,7 @@
   </inertial>
 </link>
+<gazebo reference="5th_link">
+  <material>Gazebo/Grey</material>
+</gazebo>
 <joint name="5th_to_6th" type="revolute">
   <parent link="5th_link"/>
@@ -171,5 +197,5 @@
   <axis xyz="1 0 0"/>
   <dynamics damping="0.7"/>
-  <limit lower="-1.5" upper="1.5" effort="0" velocity="0"/>
+  <limit lower="-1.5" upper="1.5" effort="0.5" velocity="6.0"/>
 </joint>
 <transmission name="5th_trans">
@@ -179,5 +205,5 @@
     </joint>
     <actuator name="5th_motor">
-       <hardwareInterface>hardware_interface/EffortJointInterface</hardwareInterface>
+      <hardwareInterface>hardware_interface/EffortJointInterface</hardwareInterface>
        <mechanismReduction>1</mechanismReduction>
     </actuator>
@@ -188,4 +214,5 @@
       <mesh filename="package://kyun_description/mesh/frame13.stl" scale="0.001 0.001 0.001"/>
     </geometry>
+    <material name="white"/>
   </visual>
   <collision>
@@ -199,4 +226,7 @@
   </inertial>
 </link>
+<gazebo reference="6th_link">
+  <material>Gazebo/white</material>
+</gazebo>
 <gazebo>
   <plugin name="gazebo_ros_control" filename="libgazebo_ros_control.so">
