Commit message: rename

File: kyun_description/urdf/kyun.xacro (robot description, xacro)
@@ -1,72 +1,125 @@
 <?xml version="1.0"?>
-<robot name="kyun" xmlns:xacro="http://ros.org/wiki/xacro">
-  <link name="world"/>
-  <joint name="world_to_base" type="fixed">
-    <origin xyz="0 0 0.0465"/>
-    <parent link="world"/>
-    <child link="base_link"/>
-  </joint>
-  <link name="base_link">
-    <visual>
-      <geometry>
-        <mesh filename="package://kyun_description/mesh/servo01.stl" scale="0.001 0.001 0.001"/>
-        <origin xyz="0 0 0.0465"/>
-      </geometry>
-    </visual>
-    <collision>
-      <geometry>
-        <mesh filename="package://kyun_description/mesh/servo01.stl" scale="0.001 0.001 0.001"/>
-        <origin xyz="0 0 0.0465"/>
-      </geometry>
-    </collision>
-    <inertial>
-      <mass value="0.0572"/>
-      <inertia ixx="0.00093819916" ixy="0" ixz="0" iyy="0.00158169916" iyz="0" izz="0.001417845"/>
-    </inertial>
-  </link>
-  <joint name="base_to_2nd" type="continuous">
-    <parent link="base_link"/>
-    <child link="2nd_link"/>
-    <origin xyz="0 0 0" rpy="0 0 0"/>
-    <axis xyz="0 0 1"/>
-    <dynamics damping="0.1"/>
-  </joint>
+<robot name="kyun" xmlns:xacro="http://www.ros.org/wiki/xacro">
+<material name="gray">
+  <color rgba="0.5 0.5 0.5 2.5"/>
+</material>
+<material name="white">
+  <color rgba="1.0 1.0 1.0 1"/>
+</material>
+<link name="world"/>
+<joint name="world_to_base" type="fixed">
+  <origin xyz="0 0 0.0465"/>
+  <parent link="world"/>
+  <child link="base_link"/>
+</joint>
+<link name="base_link">
+  <visual>
+    <geometry>
+      <mesh filename="package://kyun_description/mesh/servo01.stl" scale="0.001 0.001 0.001"/>
+      <origin xyz="0 0 0.0465"/>
+    </geometry>
+    <material name="gray"/>
+  </visual>
+  <collision>
+    <geometry>
+      <mesh filename="package://kyun_description/mesh/servo01.stl" scale="0.001 0.001 0.001"/>
+      <origin xyz="0 0 0.0465"/>
+    </geometry>
+  </collision>
+  <inertial>
+    <mass value="0.0572"/>
+    <inertia ixx="0.00093819916" ixy="0" ixz="0" iyy="0.00158169916" iyz="0" izz="0.001417845"/>
+  </inertial>
+</link>
+<gazebo reference="base_link">
+  <material>Gazebo/Grey</material>
+</gazebo>
+<joint name="base_to_2nd" type="revolute">
+  <parent link="base_link"/>
+  <child link="2nd_link"/>
+  <origin xyz="0 0 0" rpy="0 0 0"/>
+  <axis xyz="0 0 1"/>
+  <dynamics damping="0.7"/>
+  <limit lower="-1.5" upper="1.5" effort="0.5" velocity="6.0"/>
+</joint>
+<transmission name="base_trans">
+    <type>transmission_interface/SimpleTransmission</type>
+    <joint name="base_to_2nd">
+      <hardwareInterface>hardware_interface/EffortJointInterface</hardwareInterface>
+    </joint>
+    <actuator name="base_motor">
+      <hardwareInterface>hardware_interface/EffortJointInterface</hardwareInterface>
+      <mechanismReduction>1</mechanismReduction>
+    </actuator>
+</transmission>
 <link name="2nd_link">
   <visual>
     <geometry>
       <mesh filename="package://kyun_description/mesh/frame12.stl" scale="0.001 0.001 0.001"/>
-    </geometry>
+      <origin xyz="0 0 0"/>
+    </geometry>
+    <material name="grey"/>
   </visual>
   <collision>
     <geometry>
       <mesh filename="package://kyun_description/mesh/frame12.stl" scale="0.001 0.001 0.001"/>
-    </geometry>
-  </collision>
-</link>
-<joint name="2nd_to_3rd" type="continuous">
+      <origin xyz="0 0 0"/>
+    </geometry>
+  </collision>
+  <inertial>
+    <mass value="0.0228"/>
+    <inertia ixx="0.0012587" ixy="0" ixz="0" iyy="0.0009052" iyz="0" izz="0.0010677"/>
+  </inertial>
+</link>
+<gazebo reference="2nd_link">
+  <material>Gazebo/Grey</material>
+</gazebo>
+<joint name="2nd_to_3rd" type="revolute">
   <parent link="2nd_link"/>
   <child link="3rd_link"/>
   <origin xyz="-0.00963 0.019 0.05" rpy="0 0 0"/>
   <axis xyz="0 1 0"/>
-  <dynamics damping="0.1"/>
-</joint>
+  <dynamics damping="0.7"/>
+  <limit lower="-1.5" upper="1.5" effort="0.5" velocity="6.0"/>
+</joint>
+<transmission name="2nd_trans">
+    <type>transmission_interface/SimpleTransmission</type>
+    <joint name="2nd_to_3rd">
+      <hardwareInterface>hardware_interface/EffortJointInterface</hardwareInterface>
+    </joint>
+    <actuator name="2nd_motor">
+      <hardwareInterface>hardware_interface/EffortJointInterface</hardwareInterface>
+      <mechanismReduction>1</mechanismReduction>
+    </actuator>
+</transmission>
 <link name="3rd_link">
   <visual>
     <geometry>
       <mesh filename="package://kyun_description/mesh/servo02.stl" scale="0.001 0.001 0.001"/>
-    </geometry>
+      <origin xyz="0 0 0"/>
+    </geometry>
+    <material name="grey"/>
   </visual>
   <collision>
     <geometry>
       <mesh filename="package://kyun_description/mesh/servo02.stl" scale="0.001 0.001 0.001"/>
-    </geometry>
-  </collision>
-</link>
-<joint name="3rd_to_4th" type="continuous">
+      <origin xyz="0 0 0"/>
+    </geometry>
+  </collision>
+  <inertial>
+    <mass value="0.0638"/>
+    <inertia ixx="0.0021267" ixy="0" ixz="0" iyy="0.0020277" iyz="0" izz="0.0011317"/>
+  </inertial>
+</link>
+<gazebo reference="3rd_link">
+  <material>Gazebo/Grey</material>
+</gazebo>
+<joint name="3rd_to_4th" type="revolute">
   <parent link="3rd_link"/>
   <child link="4th_link"/>
   <origin xyz="0.019 -0.018 0.06075" rpy="0 0 0"/>
   <axis xyz="1 0 0"/>
-  <dynamics damping="0.1"/>
+  <dynamics damping="0.7"/>
+  <limit lower="-1.5" upper="1.5" effort="0.5" velocity="6.0"/>
 </joint>
 <transmission name="3rd_trans">
@@ -76,6 +129,6 @@
     </joint>
     <actuator name="3rd_motor">
-       <hardwareInterface>hardware_interface/EffortJointInterface</hardwareInterface>
-       <mechanismReduction>1</mechanismReduction>
+      <hardwareInterface>hardware_interface/EffortJointInterface</hardwareInterface>
+      <mechanismReduction>1</mechanismReduction>
     </actuator>
 </transmission>
@@ -85,4 +138,5 @@
       <mesh filename="package://kyun_description/mesh/servo03.stl" scale="0.001 0.001 0.001"/>
     </geometry>
+    <material name="grey"/>
   </visual>
   <collision>
@@ -91,11 +145,19 @@
     </geometry>
   </collision>
-</link>
-<joint name="4th_to_5th" type="continuous">
+  <inertial>
+    <mass value="0.099806"/>
+    <inertia ixx="0.0028791" ixy="0" ixz="0" iyy="0.0028648" iyz="0" izz="0.0021805"/>
+  </inertial>
+</link>
+<gazebo reference="4th_link">
+  <material>Gazebo/Grey</material>
+</gazebo>
+<joint name="4th_to_5th" type="revolute">
   <parent link="4th_link"/>
   <child link="5th_link"/>
   <origin xyz="-0.019 -0.02 0.024" rpy="0 0 0"/>
   <axis xyz="0 1 0"/>
-  <dynamics damping="0.1"/>
+  <dynamics damping="0.7"/>
+  <limit lower="-1.5" upper="1.5" effort="0.5" velocity="6.0"/>
 </joint>
 <transmission name="4th_trans">
@@ -105,6 +167,6 @@
     </joint>
     <actuator name="4th_motor">
-       <hardwareInterface>hardware_interface/EffortJointInterface</hardwareInterface>
-       <mechanismReduction>1</mechanismReduction>
+      <hardwareInterface>hardware_interface/EffortJointInterface</hardwareInterface>
+      <mechanismReduction>1</mechanismReduction>
     </actuator>
 </transmission>
@@ -114,4 +176,5 @@
       <mesh filename="package://kyun_description/mesh/servo04.stl" scale="0.001 0.001 0.001"/>
     </geometry>
+    <material name="grey"/>
   </visual>
   <collision>
@@ -120,11 +183,19 @@
     </geometry>
   </collision>
-</link>
-<joint name="5th_to_6th" type="continuous">
+  <inertial>
+    <mass value="0.063759"/>
+    <inertia ixx="0.0020277" ixy="0" ixz="0" iyy="0.0021267" iyz="0" izz="0.0011317"/>
+  </inertial>
+</link>
+<gazebo reference="5th_link">
+  <material>Gazebo/Grey</material>
+</gazebo>
+<joint name="5th_to_6th" type="revolute">
   <parent link="5th_link"/>
   <child link="6th_link"/>
   <origin xyz="0.0205 0.02 0.06075" rpy="0 0 0"/>
   <axis xyz="1 0 0"/>
-  <dynamics damping="0.1"/>
+  <dynamics damping="0.7"/>
+  <limit lower="-1.5" upper="1.5" effort="0.5" velocity="6.0"/>
 </joint>
 <transmission name="5th_trans">
@@ -134,5 +205,5 @@
     </joint>
     <actuator name="5th_motor">
-       <hardwareInterface>hardware_interface/EffortJointInterface</hardwareInterface>
+      <hardwareInterface>hardware_interface/EffortJointInterface</hardwareInterface>
        <mechanismReduction>1</mechanismReduction>
     </actuator>
@@ -143,4 +214,5 @@
       <mesh filename="package://kyun_description/mesh/frame13.stl" scale="0.001 0.001 0.001"/>
     </geometry>
+    <material name="white"/>
   </visual>
   <collision>
@@ -149,11 +221,18 @@
     </geometry>
   </collision>
-</link>
-  <gazebo>
-    <plugin name="gazebo_ros_control" filename="libgazebo_ros_control.so">
-      <robotNamespace>/kyun</robotNamespace>
-      <robotSimType>gazebo_ros_control/DefaultRobotHWSim</robotSimType>
-      <legacyModeNS>true</legacyModeNS>
-    </plugin>
-  </gazebo>
+  <inertial>
+    <mass value="0.059571"/>
+    <inertia ixx="0.0011416" ixy="0" ixz="0" iyy="0.0011103" iyz="0" izz="0.0020421"/>
+  </inertial>
+</link>
+<gazebo reference="6th_link">
+  <material>Gazebo/white</material>
+</gazebo>
+<gazebo>
+  <plugin name="gazebo_ros_control" filename="libgazebo_ros_control.so">
+    <robotNamespace>/kyun</robotNamespace>
+    <robotSimType>gazebo_ros_control/DefaultRobotHWSim</robotSimType>
+    <legacyModeNS>true</legacyModeNS>
+  </plugin>
+</gazebo>
 </robot>

Commit message: add arm_controller to dynemixel_workbench

File: kyun_description/urdf/kyun.xacro (robot description, xacro)
@@ -46,8 +46,8 @@
     <type>transmission_interface/SimpleTransmission</type>
     <joint name="base_to_2nd">
-      <hardwareInterface>hardware_interface/EffortJointInterface</hardwareInterface>
+      <hardwareInterface>hardware_interface/PositionJointInterface</hardwareInterface>
     </joint>
     <actuator name="base_motor">
-      <hardwareInterface>hardware_interface/EffortJointInterface</hardwareInterface>
+      <hardwareInterface>hardware_interface/PositionJointInterface</hardwareInterface>
       <mechanismReduction>1</mechanismReduction>
     </actuator>
@@ -86,8 +86,8 @@
     <type>transmission_interface/SimpleTransmission</type>
     <joint name="2nd_to_3rd">
-      <hardwareInterface>hardware_interface/EffortJointInterface</hardwareInterface>
+      <hardwareInterface>hardware_interface/PositionJointInterface</hardwareInterface>
     </joint>
     <actuator name="2nd_motor">
-      <hardwareInterface>hardware_interface/EffortJointInterface</hardwareInterface>
+      <hardwareInterface>hardware_interface/PositionJointInterface</hardwareInterface>
       <mechanismReduction>1</mechanismReduction>
     </actuator>
@@ -126,8 +126,8 @@
     <type>transmission_interface/SimpleTransmission</type>
     <joint name="3rd_to_4th">
-      <hardwareInterface>hardware_interface/EffortJointInterface</hardwareInterface>
+      <hardwareInterface>hardware_interface/PositionJointInterface</hardwareInterface>
     </joint>
     <actuator name="3rd_motor">
-      <hardwareInterface>hardware_interface/EffortJointInterface</hardwareInterface>
+      <hardwareInterface>hardware_interface/PositionJointInterface</hardwareInterface>
       <mechanismReduction>1</mechanismReduction>
     </actuator>
@@ -164,8 +164,8 @@
     <type>transmission_interface/SimpleTransmission</type>
     <joint name="4th_to_5th">
-      <hardwareInterface>hardware_interface/EffortJointInterface</hardwareInterface>
+      <hardwareInterface>hardware_interface/PositionJointInterface</hardwareInterface>
     </joint>
     <actuator name="4th_motor">
-      <hardwareInterface>hardware_interface/EffortJointInterface</hardwareInterface>
+      <hardwareInterface>hardware_interface/PositionJointInterface</hardwareInterface>
       <mechanismReduction>1</mechanismReduction>
     </actuator>
@@ -202,8 +202,8 @@
     <type>transmission_interface/SimpleTransmission</type>
     <joint name="5th_to_6th">
-      <hardwareInterface>hardware_interface/EffortJointInterface</hardwareInterface>
+      <hardwareInterface>hardware_interface/PositionJointInterface</hardwareInterface>
     </joint>
     <actuator name="5th_motor">
-      <hardwareInterface>hardware_interface/EffortJointInterface</hardwareInterface>
+      <hardwareInterface>hardware_interface/PositionJointInterface</hardwareInterface>
        <mechanismReduction>1</mechanismReduction>
     </actuator>
@@ -236,3 +236,8 @@
   </plugin>
 </gazebo>
+<gazebo>
+  <plugin name="joint_state_publisher" filename="libgazebo_ros_joint_state_publisher.so">
+    <jointName>base_to_2nd, 2nd_to_3rd, 3rd_to_4th, 4th_to_5th, 5th_to_6th</jointName>
+  </plugin>
+</gazebo>
 </robot>

File: kyun_real_description_sdk/urdf/kyun_real.xacro (robot description, xacro)
@@ -1,4 +1,4 @@
 <?xml version="1.0"?>
-<robot name="kyun_real" xmlns:xacro="http://www.ros.org/wiki/xacro">
+<robot name="kyun" xmlns:xacro="http://www.ros.org/wiki/xacro">
 <material name="gray">
   <color rgba="0.5 0.5 0.5 2.5"/>
@@ -16,5 +16,5 @@
   <visual>
     <geometry>
-      <mesh filename="package://kyun_real_description/mesh/servo01.stl" scale="0.001 0.001 0.001"/>
+      <mesh filename="package://kyun_real_description_sdk/mesh/servo01.stl" scale="0.001 0.001 0.001"/>
       <origin xyz="0 0 0.0465"/>
     </geometry>
@@ -23,5 +23,5 @@
   <collision>
     <geometry>
-      <mesh filename="package://kyun_real_description/mesh/servo01.stl" scale="0.001 0.001 0.001"/>
+      <mesh filename="package://kyun_real_description_sdk/mesh/servo01.stl" scale="0.001 0.001 0.001"/>
       <origin xyz="0 0 0.0465"/>
     </geometry>
@@ -53,12 +53,12 @@
   <visual>
     <geometry>
-      <mesh filename="package://kyun_real_description/mesh/frame12.stl" scale="0.001 0.001 0.001"/>
-      <origin xyz="0 0 0"/>
-    </geometry>
-    <material name="grey"/>
-  </visual>
-  <collision>
-    <geometry>
-      <mesh filename="package://kyun_real_description/mesh/frame12.stl" scale="0.001 0.001 0.001"/>
+      <mesh filename="package://kyun_real_description_sdk/mesh/frame12.stl" scale="0.001 0.001 0.001"/>
+      <origin xyz="0 0 0"/>
+    </geometry>
+    <material name="grey"/>
+  </visual>
+  <collision>
+    <geometry>
+      <mesh filename="package://kyun_real_description_sdk/mesh/frame12.stl" scale="0.001 0.001 0.001"/>
       <origin xyz="0 0 0"/>
     </geometry>
@@ -90,12 +90,12 @@
   <visual>
     <geometry>
-      <mesh filename="package://kyun_real_description/mesh/servo02.stl" scale="0.001 0.001 0.001"/>
-      <origin xyz="0 0 0"/>
-    </geometry>
-    <material name="grey"/>
-  </visual>
-  <collision>
-    <geometry>
-      <mesh filename="package://kyun_real_description/mesh/servo02.stl" scale="0.001 0.001 0.001"/>
+      <mesh filename="package://kyun_real_description_sdk/mesh/servo02.stl" scale="0.001 0.001 0.001"/>
+      <origin xyz="0 0 0"/>
+    </geometry>
+    <material name="grey"/>
+  </visual>
+  <collision>
+    <geometry>
+      <mesh filename="package://kyun_real_description_sdk/mesh/servo02.stl" scale="0.001 0.001 0.001"/>
       <origin xyz="0 0 0"/>
     </geometry>
@@ -127,11 +127,11 @@
   <visual>
     <geometry>
-      <mesh filename="package://kyun_description/mesh/servo03.stl" scale="0.001 0.001 0.001"/>
-    </geometry>
-    <material name="grey"/>
-  </visual>
-  <collision>
-    <geometry>
-      <mesh filename="package://kyun_description/mesh/servo03.stl" scale="0.001 0.001 0.001"/>
+      <mesh filename="package://kyun_real_description_sdk/mesh/servo03.stl" scale="0.001 0.001 0.001"/>
+    </geometry>
+    <material name="grey"/>
+  </visual>
+  <collision>
+    <geometry>
+      <mesh filename="package://kyun_real_description_sdk/mesh/servo03.stl" scale="0.001 0.001 0.001"/>
     </geometry>
   </collision>
@@ -162,11 +162,11 @@
   <visual>
     <geometry>
-      <mesh filename="package://kyun_description/mesh/servo04.stl" scale="0.001 0.001 0.001"/>
-    </geometry>
-    <material name="grey"/>
-  </visual>
-  <collision>
-    <geometry>
-      <mesh filename="package://kyun_description/mesh/servo04.stl" scale="0.001 0.001 0.001"/>
+      <mesh filename="package://kyun_real_description_sdk/mesh/servo04.stl" scale="0.001 0.001 0.001"/>
+    </geometry>
+    <material name="grey"/>
+  </visual>
+  <collision>
+    <geometry>
+      <mesh filename="package://kyun_real_description_sdk/mesh/servo04.stl" scale="0.001 0.001 0.001"/>
     </geometry>
   </collision>
@@ -197,5 +197,5 @@
   <visual>
     <geometry>
-      <mesh filename="package://kyun_description/mesh/frame13.stl" scale="0.001 0.001 0.001"/>
+      <mesh filename="package://kyun_real_description_sdk/mesh/frame13.stl" scale="0.001 0.001 0.001"/>
     </geometry>
     <material name="white"/>
@@ -203,5 +203,5 @@
   <collision>
     <geometry>
-      <mesh filename="package://kyun_description/mesh/frame13.stl" scale="0.001 0.001 0.001"/>
+      <mesh filename="package://kyun_real_description_sdk/mesh/frame13.stl" scale="0.001 0.001 0.001"/>
     </geometry>
   </collision>
