Commit message: rename

File: kyun_description/urdf/kyun.xacro (robot description, xacro)
@@ -23,5 +23,5 @@
   <collision>
     <geometry>
-      <mesh filename="package://kyun_description/mesh/servo01.stl" scale="0.001 0.001 0.001"/>
+      <mesh filename="package://kyun_description/mesh/servo01.stl" scale="0.0009 0.0009 0.0009"/>
       <origin xyz="0 0 0.0465"/>
     </geometry>
@@ -35,7 +35,7 @@
   <material>Gazebo/Grey</material>
 </gazebo>
-<joint name="base_to_2nd" type="revolute">
+<joint name="base_to_second" type="revolute">
   <parent link="base_link"/>
-  <child link="2nd_link"/>
+  <child link="second_link"/>
   <origin xyz="0 0 0" rpy="0 0 0"/>
   <axis xyz="0 0 1"/>
@@ -45,5 +45,5 @@
 <transmission name="base_trans">
     <type>transmission_interface/SimpleTransmission</type>
-    <joint name="base_to_2nd">
+    <joint name="base_to_second">
       <hardwareInterface>hardware_interface/PositionJointInterface</hardwareInterface>
     </joint>
@@ -53,5 +53,5 @@
     </actuator>
 </transmission>
-<link name="2nd_link">
+<link name="second_link">
   <visual>
     <geometry>
@@ -63,5 +63,5 @@
   <collision>
     <geometry>
-      <mesh filename="package://kyun_description/mesh/frame12.stl" scale="0.001 0.001 0.001"/>
+      <mesh filename="package://kyun_description/mesh/frame12.stl" scale="0.0009 0.0009 0.0009"/>
       <origin xyz="0 0 0"/>
     </geometry>
@@ -72,10 +72,10 @@
   </inertial>
 </link>
-<gazebo reference="2nd_link">
-  <material>Gazebo/Grey</material>
-</gazebo>
-<joint name="2nd_to_3rd" type="revolute">
-  <parent link="2nd_link"/>
-  <child link="3rd_link"/>
+<gazebo reference="second_link">
+  <material>Gazebo/Grey</material>
+</gazebo>
+<joint name="second_to_third" type="revolute">
+  <parent link="second_link"/>
+  <child link="third_link"/>
   <origin xyz="-0.00963 0.019 0.05" rpy="0 0 0"/>
   <axis xyz="0 1 0"/>
@@ -83,15 +83,15 @@
   <limit lower="-1.5" upper="1.5" effort="0.5" velocity="6.0"/>
 </joint>
-<transmission name="2nd_trans">
-    <type>transmission_interface/SimpleTransmission</type>
-    <joint name="2nd_to_3rd">
-      <hardwareInterface>hardware_interface/PositionJointInterface</hardwareInterface>
-    </joint>
-    <actuator name="2nd_motor">
-      <hardwareInterface>hardware_interface/PositionJointInterface</hardwareInterface>
-      <mechanismReduction>1</mechanismReduction>
-    </actuator>
-</transmission>
-<link name="3rd_link">
+<transmission name="second_trans">
+    <type>transmission_interface/SimpleTransmission</type>
+    <joint name="second_to_third">
+      <hardwareInterface>hardware_interface/PositionJointInterface</hardwareInterface>
+    </joint>
+    <actuator name="second_motor">
+      <hardwareInterface>hardware_interface/PositionJointInterface</hardwareInterface>
+      <mechanismReduction>1</mechanismReduction>
+    </actuator>
+</transmission>
+<link name="third_link">
   <visual>
     <geometry>
@@ -103,5 +103,5 @@
   <collision>
     <geometry>
-      <mesh filename="package://kyun_description/mesh/servo02.stl" scale="0.001 0.001 0.001"/>
+      <mesh filename="package://kyun_description/mesh/servo02.stl" scale="0.0009 0.0009 0.0009"/>
       <origin xyz="0 0 0"/>
     </geometry>
@@ -112,10 +112,10 @@
   </inertial>
 </link>
-<gazebo reference="3rd_link">
-  <material>Gazebo/Grey</material>
-</gazebo>
-<joint name="3rd_to_4th" type="revolute">
-  <parent link="3rd_link"/>
-  <child link="4th_link"/>
+<gazebo reference="third_link">
+  <material>Gazebo/Grey</material>
+</gazebo>
+<joint name="third_to_fourth" type="revolute">
+  <parent link="third_link"/>
+  <child link="fourth_link"/>
   <origin xyz="0.019 -0.018 0.06075" rpy="0 0 0"/>
   <axis xyz="1 0 0"/>
@@ -123,15 +123,15 @@
   <limit lower="-1.5" upper="1.5" effort="0.5" velocity="6.0"/>
 </joint>
-<transmission name="3rd_trans">
-    <type>transmission_interface/SimpleTransmission</type>
-    <joint name="3rd_to_4th">
-      <hardwareInterface>hardware_interface/PositionJointInterface</hardwareInterface>
-    </joint>
-    <actuator name="3rd_motor">
-      <hardwareInterface>hardware_interface/PositionJointInterface</hardwareInterface>
-      <mechanismReduction>1</mechanismReduction>
-    </actuator>
-</transmission>
-<link name="4th_link">
+<transmission name="third_trans">
+    <type>transmission_interface/SimpleTransmission</type>
+    <joint name="third_to_fourth">
+      <hardwareInterface>hardware_interface/PositionJointInterface</hardwareInterface>
+    </joint>
+    <actuator name="third_motor">
+      <hardwareInterface>hardware_interface/PositionJointInterface</hardwareInterface>
+      <mechanismReduction>1</mechanismReduction>
+    </actuator>
+</transmission>
+<link name="fourth_link">
   <visual>
     <geometry>
@@ -142,5 +142,5 @@
   <collision>
     <geometry>
-      <mesh filename="package://kyun_description/mesh/servo03.stl" scale="0.001 0.001 0.001"/>
+      <mesh filename="package://kyun_description/mesh/servo03.stl" scale="0.0009 0.0009 0.0009"/>
     </geometry>
   </collision>
@@ -150,10 +150,10 @@
   </inertial>
 </link>
-<gazebo reference="4th_link">
-  <material>Gazebo/Grey</material>
-</gazebo>
-<joint name="4th_to_5th" type="revolute">
-  <parent link="4th_link"/>
-  <child link="5th_link"/>
+<gazebo reference="fourth_link">
+  <material>Gazebo/Grey</material>
+</gazebo>
+<joint name="fourth_to_fifth" type="revolute">
+  <parent link="fourth_link"/>
+  <child link="fifth_link"/>
   <origin xyz="-0.019 -0.02 0.024" rpy="0 0 0"/>
   <axis xyz="0 1 0"/>
@@ -161,15 +161,15 @@
   <limit lower="-1.5" upper="1.5" effort="0.5" velocity="6.0"/>
 </joint>
-<transmission name="4th_trans">
-    <type>transmission_interface/SimpleTransmission</type>
-    <joint name="4th_to_5th">
-      <hardwareInterface>hardware_interface/PositionJointInterface</hardwareInterface>
-    </joint>
-    <actuator name="4th_motor">
-      <hardwareInterface>hardware_interface/PositionJointInterface</hardwareInterface>
-      <mechanismReduction>1</mechanismReduction>
-    </actuator>
-</transmission>
-<link name="5th_link">
+<transmission name="fourth_trans">
+    <type>transmission_interface/SimpleTransmission</type>
+    <joint name="fourth_to_fifth">
+      <hardwareInterface>hardware_interface/PositionJointInterface</hardwareInterface>
+    </joint>
+    <actuator name="fourth_motor">
+      <hardwareInterface>hardware_interface/PositionJointInterface</hardwareInterface>
+      <mechanismReduction>1</mechanismReduction>
+    </actuator>
+</transmission>
+<link name="fifth_link">
   <visual>
     <geometry>
@@ -180,5 +180,5 @@
   <collision>
     <geometry>
-      <mesh filename="package://kyun_description/mesh/servo04.stl" scale="0.001 0.001 0.001"/>
+      <mesh filename="package://kyun_description/mesh/servo04.stl" scale="0.0009 0.0009 0.0009"/>
     </geometry>
   </collision>
@@ -188,10 +188,10 @@
   </inertial>
 </link>
-<gazebo reference="5th_link">
-  <material>Gazebo/Grey</material>
-</gazebo>
-<joint name="5th_to_6th" type="revolute">
-  <parent link="5th_link"/>
-  <child link="6th_link"/>
+<gazebo reference="fifth_link">
+  <material>Gazebo/Grey</material>
+</gazebo>
+<joint name="fifth_to_sixth" type="revolute">
+  <parent link="fifth_link"/>
+  <child link="sixth_link"/>
   <origin xyz="0.0205 0.02 0.06075" rpy="0 0 0"/>
   <axis xyz="1 0 0"/>
@@ -199,15 +199,15 @@
   <limit lower="-1.5" upper="1.5" effort="0.5" velocity="6.0"/>
 </joint>
-<transmission name="5th_trans">
-    <type>transmission_interface/SimpleTransmission</type>
-    <joint name="5th_to_6th">
-      <hardwareInterface>hardware_interface/PositionJointInterface</hardwareInterface>
-    </joint>
-    <actuator name="5th_motor">
-      <hardwareInterface>hardware_interface/PositionJointInterface</hardwareInterface>
+<transmission name="fifth_trans">
+    <type>transmission_interface/SimpleTransmission</type>
+    <joint name="fifth_to_sixth">
+      <hardwareInterface>hardware_interface/PositionJointInterface</hardwareInterface>
+    </joint>
+    <actuator name="fifth_motor">
+      <hardwareInterface>hardware_interface/EPositionJointInterface</hardwareInterface>
        <mechanismReduction>1</mechanismReduction>
     </actuator>
 </transmission>
-<link name="6th_link">
+<link name="sixth_link">
   <visual>
     <geometry>
@@ -218,5 +218,5 @@
   <collision>
     <geometry>
-      <mesh filename="package://kyun_description/mesh/frame13.stl" scale="0.001 0.001 0.001"/>
+      <mesh filename="package://kyun_description/mesh/frame13.stl" scale="0.0009 0.0009 0.0009"/>
     </geometry>
   </collision>
@@ -226,5 +226,5 @@
   </inertial>
 </link>
-<gazebo reference="6th_link">
+<gazebo reference="sixth_link">
   <material>Gazebo/white</material>
 </gazebo>
@@ -235,8 +235,6 @@
     <legacyModeNS>true</legacyModeNS>
   </plugin>
-</gazebo>
-<gazebo>
   <plugin name="joint_state_publisher" filename="libgazebo_ros_joint_state_publisher.so">
-    <jointName>base_to_2nd, 2nd_to_3rd, 3rd_to_4th, 4th_to_5th, 5th_to_6th</jointName>
+    <jointName>base_to_second, second_to_third, third_to_fourth, fourth_to_fifth, fifth_to_sixth</jointName>
   </plugin>
 </gazebo>
